Commit message: add code

File: data/franka_panda/panda_longer_finger_mplib.urdf (robot description, URDF)
Before this commit: robot panda, 17 links, 16 joints
Links:
- link finger_left_tip: geometry collision mesh filename=meshes/visual/digit_gel_only.STL; visual mesh filename=meshes/visual/digit_gel_only.STL
- link finger_right_tip: geometry collision mesh filename=meshes/visual/digit_gel_only.STL; visual mesh filename=meshes/visual/digit_gel_only.STL
- link panda_hand: geometry collision mesh filename=meshes/collision/hand.obj; visual mesh filename=meshes/visual/hand.obj
- link panda_leftfinger: geometry collision mesh filename=meshes/collision/longer_finger_v2.obj; visual mesh filename=meshes/visual/longer_finger_v2.obj
- link panda_link0: geometry collision mesh filename=meshes/collision/link0.obj; visual mesh filename=meshes/collision/link0.obj
- link panda_link1: geometry collision mesh filename=meshes/collision/link1.obj; visual mesh filename=meshes/visual/link1.obj
- link panda_link2: geometry collision mesh filename=meshes/collision/link2.obj; visual mesh filename=meshes/visual/link2.obj
- link panda_link3: geometry collision mesh filename=meshes/collision/link3.obj; visual mesh filename=meshes/visual/link3.obj
- link panda_link4: geometry collision mesh filename=meshes/collision/link4.obj; visual mesh filename=meshes/visual/link4.obj
- link panda_link5: geometry collision mesh filename=meshes/collision/link5.obj; visual mesh filename=meshes/visual/link5.obj
- link panda_link6: geometry collision mesh filename=meshes/collision/link6.obj; visual mesh filename=meshes/visual/link6.obj
- link panda_link7: geometry collision mesh filename=meshes/collision/link7.obj; visual mesh filename=meshes/collision/link7.obj
- link panda_rightfinger: geometry collision mesh filename=meshes/collision/longer_finger_v2.obj; visual mesh filename=meshes/visual/longer_finger_v2.obj
